Commit message: adding wheels
created two wheels as links with their joints. The y have basic configurations

File: src/udacity_bot/urdf/udacity_bot.xacro (robot description, xacro)
@@ -55,3 +55,67 @@
     </visual>
   </link>
+  <link name='right_wheel'>
+	  <pose>0 0 0.1 0 0 0</pose>
+	  <inertial>
+	      <mass value="5.0"/>
+	      <origin xyz="0 0 0" rpy="0 1.5707 1.5707 "/>
+	      <inertia
+		  ixx="0.1" ixy="0" ixz="0"
+		  iyy="0.1" iyz="0"
+		  izz="0.1"
+	      />
+	    </inertial>
+	    <collision name='right_wheel_collision'>
+	      <origin xyz="0 0 0" rpy=" 0 1.5707 1.5707"/>
+	      <geometry>
+		<cylinder radius="0.1" length="0.05"/>
+	      </geometry>
+	    </collision>
+	    <visual name='right_wheel_visual'>
+	      <origin xyz="0 0 0" rpy=" 0 1.5707 1.5707"/>
+	      <geometry>
+		<cylinder radius="0.1" length="0.05"/>
+	      </geometry>
+	    </visual>
+  </link>
+  <link name='left_wheel'>
+	  <pose>0 0 0.1 0 0 0</pose>
+	  <inertial>
+	      <mass value="5.0"/>
+	      <origin xyz="0 0 0" rpy="0 1.5707 1.5707"/>
+	      <inertia
+		  ixx="0.1" ixy="0" ixz="0"
+		  iyy="0.1" iyz="0"
+		  izz="0.1"
+	      />
+	    </inertial>
+	    <collision name='left_wheel_collision'>
+	      <origin xyz="0 0 0" rpy=" 0 1.5707 1.5707"/>
+	      <geometry>
+		<cylinder radius="0.1" length="0.05"/>
+	      </geometry>
+	    </collision>
+	    <visual name='left_wheel_visual'>
+	      <origin xyz="0 0 0" rpy=" 0 1.5707 1.5707"/>
+	      <geometry>
+		<cylinder radius="0.1" length="0.05"/>
+	      </geometry>
+	    </visual>
+  </link>
+  <joint type="continuous" name="left_wheel_hinge">
+	    <origin xyz="0 0.15 0" rpy="0 0 0"/>
+	    <child link="left_wheel"/>
+	    <parent link="chassis"/>
+	    <axis xyz="0 1 0" rpy="0 0 0"/>
+	    <limit effort="10000" velocity="1000"/>
+	    <dynamics damping="1.0" friction="1.0"/>
+  </joint>
+  <joint type="continuous" name="right_wheel_hinge">
+	    <origin xyz="0 -0.15 0" rpy="0 0 0"/>
+	    <child link="right_wheel"/>
+	    <parent link="chassis"/>
+	    <axis xyz="0 1 0" rpy="0 0 0"/>
+	    <limit effort="10000" velocity="1000"/>
+	    <dynamics damping="1.0" friction="1.0"/>
+  </joint>
 </robot>

Commit message: camera and hokuyo
added link and joints of sensor. hokuyo has mesh file attached

File: src/udacity_bot/urdf/udacity_bot.xacro (robot description, xacro)
@@ -119,3 +119,61 @@
 	    <dynamics damping="1.0" friction="1.0"/>
   </joint>
+  <link name='camera'>
+	  <pose>0 0 0.1 0 0 0</pose>
+	  <inertial>
+	      <mass value="0.1"/>
+	      <origin xyz="0 0 0" rpy="0 0 0"/>
+	      <inertia
+		  ixx="1e-6" ixy="0" ixz="0"
+		  iyy="1e-6" iyz="0"
+		  izz="1e-6"
+	      />
+	    </inertial>
+	    <collision name='camera_collision'>
+	      <origin xyz="0 0 0" rpy=" 0 0 0"/>
+	      <geometry>
+		<box size="0.05 0.05 0.05"/>
+	      </geometry>
+	    </collision>
+	    <visual name='camera_visual'>
+	      <origin xyz="0 0 0" rpy=" 0 0 0"/>
+	      <geometry>
+		<box size="0.05 0.05 0.05"/>
+	      </geometry>
+	    </visual>
+  </link>
+  <joint type="fixed" name="camera_joint">
+	    <origin xyz="0.2 0 0" rpy="0 0 0"/>
+	    <child link="camera"/>
+	    <parent link="chassis"/>
+  </joint>
+  <link name='hokuyo'>
+	  <pose>0 0 0.1 0 0 0</pose>
+	  <inertial>
+	      <mass value="0.1"/>
+	      <origin xyz="0 0 0" rpy="0 0 0"/>
+	      <inertia
+		  ixx="1e-6" ixy="0" ixz="0"
+		  iyy="1e-6" iyz="0"
+		  izz="1e-6"
+	      />
+	    </inertial>
+	    <collision name='hokuyo_collision'>
+	      <origin xyz="0 0 0" rpy=" 0 0 0"/>
+	      <geometry>
+		<box size="0.01 0.01 0.01"/>
+	      </geometry>
+	    </collision>
+	    <visual name='hokuyo_visual'>
+	      <origin xyz="0 0 0" rpy=" 0 0 0"/>
+	      <geometry>
+		<mesh filename="$(find udacity_bot)/meshes/hokuyo.dae"/>
+	      </geometry>
+	    </visual>
+  </link>
+  <joint type="fixed" name="hokuyo_joint">
+	    <origin xyz="0.15 0 0.1" rpy="0 0 0"/>
+	    <child link="hokuyo"/>
+	    <parent link="chassis"/>
+  </joint>
 </robot>
